File: eaglefiles/crawler2body.brd (EAGLE design)
At the start: 69 x 38 mm, 40 parts, among them J2 USB-AB-MICROB-2, U1 MCP73831, U2 PCA9685, U3 FT232R, U5 LM3671MF-3.3/NOPB

Commit message: Review: crawler2body
Parts:
- added R5: 1k, SparkFun-Resistors:0603
- added R7: 3k, SparkFun-Resistors:0603
- added S1: (no value), switch-omron:B3F-10XX
Connections:
- removed net CTS: U3.11
- removed net DCD: U3.10
- removed net DSR: U3.9
- removed net DTR: U3.2
- removed net N$20: U$1.P$2
- removed net N$21: U$1.P$3
- removed net N$22: U$1.P$4
- removed net N$23: U$1.P$5
- removed net N$24: U$1.P$6
- removed net N$25: U$1.P$7
- removed net N$26: U$1.P$8
- removed net N$27: U$1.P$9
- removed net N$28: U$1.P$10
- removed net N$29: U$1.P$11
- removed net N$30: U$1.P$12
- removed net N$31: U$1.P$13
- removed net N$32: U$1.P$14
- removed net N$33: U$1.P$15
- removed net N$34: U$1.P$16
- removed net N$35: U$2.P$3
- removed net N$36: U$2.P$4
- removed net N$37: U$2.P$5
- removed net N$38: U$2.P$6
- removed net N$39: U$2.P$7
- removed net N$40: U$2.P$8
- removed net N$41: U$2.P$9
- removed net N$42: U$2.P$10
- removed net N$43: U$2.P$13
- removed net N$44: U$2.P$14
- removed net PWREN: U3.14
- removed net RI: U3.6
- removed net RTS: U3.3
- removed net SLEEP: U3.12
- removed net TXDEN: U3.13
- new net N$46: R5.1, S1.3, S1.4
- new net RESET_BTN: R5.2, R7.1, U$2.P$10
- net +3V3: now also S1.1, S1.2
- net GND: now also R7.2
Other:
- outline, holes or cut-outs redrawn
