File: eaglefiles/crawler2body.brd (EAGLE design)
At the start: 69 x 38 mm, 40 parts, among them J2 USB-AB-MICROB-2, U1 MCP73831, U2 PCA9685, U3 FT232R, U5 LM3671MF-3.3/NOPB

Commit message: review
Parts:
- moved TO_HIP02 2.00 mm to (89.0, 83.0)
- moved TO_SHOULDER02 2.00 mm to (78.0, 83.0)
- moved C9 1.12 mm to (87.6, 74.1)
- moved U$3 1.00 mm to (88.8, 69.0)
- moved C10 0.87 mm to (87.4, 63.9)
Routing:
- net V+: track 29.8 -> 36.7 mm, vias 8 -> 10
- net GND: track 26.9 -> 29.5 mm, vias 47 -> 46
- net SDA: track 49.3 -> 51.3 mm
- net SCL: track 48.3 -> 50.3 mm
- net N$16: track 21.8 -> 22.8 mm
- net N$15: track 17.8 -> 18.8 mm
- net N$13: track 21.5 -> 22.5 mm
- net N$12: track 23.1 -> 24.1 mm
- net N$11: track 24.6 -> 25.6 mm
- net N$10: track 26.5 -> 27.5 mm
- net N$14: track 14.1 -> 15.0 mm
- net N$9: track 29.1 -> 29.8 mm
- net +3V3: track 24.6 -> 25.1 mm
- added copper zone on layer 16, net GND1
- removed copper zone on layer 1, net GND1
Other:
- outline, holes or cut-outs redrawn

Commit message: review 2
Signed-off-by: Julian <julian.wingert@subtilitas.de>
Parts:
- added TP1, TP2: PTR1TP15SQ, testpad:TP15SQ
- added U$8: MF-SMDF150, fuse:MF-SMDF050
- moved JP1 1.00 mm to (78.6, 69.1)
- moved L1 0.81 mm to (111.3, 67.0)
- moved C1 0.20 mm to (107.9, 67.8)
Connections:
- removed net N$42: U$2.P$10
- new net FW_RST: TP1.TP, U$2.P$10
- new net N$46: JP2.2, U$8.1
- net +3V3: no longer U3.4
- net 3.3VFTDI: now also U3.4
- net GND: now also TP2.TP
- net USB_D+: now also J2.D+; no longer J2.D-
- net USB_D-: now also J2.D-; no longer J2.D+
- net V+: now also U$8.2; no longer JP2.2
Routing:
- net FW_RST: track 0.00 -> 13.3 mm, vias 0 -> 1
- net 3.3VFTDI: track 3.64 -> 14.0 mm
- net V_USB: track 40.9 -> 32.8 mm, vias 0 -> 2
- net N$46: track 0.00 -> 3.56 mm
- net V+: track 36.7 -> 40.0 mm, vias 10 -> 12
- net +3V3: track 25.1 -> 23.8 mm, vias 10 -> 8
- net N$1: track 3.25 -> 2.43 mm
- net GND: vias 46 -> 75

Commit message: Review-review-review Signed-off-by: Julian <julian.wingert@subtilitas.de>
Parts:
- added R5: 3k, SparkFun-Resistors:0603
- added R7: 1k, SparkFun-Resistors:0603
- JP2: device SparkFun-Connectors:JST-2-PTH -> SparkFun-Connectors:JST-2-PTH-NS
Connections:
- new net N$42: R7.2, TP2.TP
- net +3V3: now also R7.1
- net FW_RST: now also R5.2
- net GND: now also R5.1; no longer TP2.TP
Routing:
- net N$42: track 0.00 -> 2.23 mm
- net +3V3: track 23.8 -> 24.8 mm, vias 8 -> 9
Changed lines of the file:
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@@
 <setting verticaltext="up"/>
 </settings>
-<grid distance="1" unitdist="mm" unit="mm" style="lines" multiple="1" display="yes" altdistance="5" altunitdist="mil" altunit="mil"/>
+<grid distance="8" unitdist="mil" unit="mil" style="lines" multiple="1" display="yes" altdistance="5" altunitdist="mil" altunit="mil"/>
 <layers>
-<layer number="1" name="Top" color="4" fill="1" visible="no" active="yes"/>
-<layer number="2" name="Route2" color="1" fill="3" visible="no" active="yes"/>
+<layer number="1" name="Top" color="4" fill="1" visible="yes" active="yes"/>
+<layer number="2" name="Route2" color="1" fill="3" visible="yes" active="yes"/>
 <layer number="3" name="Route3" color="4" fill="3" visible="no" active="no"/>
 <layer number="4" name="Route4" color="1" fill="4" visible="no" active="no"/>
@@
 <layer number="13" name="Route13" color="4" fill="5" visible="no" active="no"/>
 <layer number="14" name="Route14" color="1" fill="6" visible="no" active="no"/>
-<layer number="15" name="Route15" color="4" fill="6" visible="no" active="yes"/>
+<layer number="15" name="Route15" color="4" fill="6" visible="yes" active="yes"/>
 <layer number="16" name="Bottom" color="1" fill="1" visible="yes" active="yes"/>
 <layer number="17" name="Pads" color="2" fill="1" visible="yes" active="yes"/>
@@
 <layer number="46" name="Milling" color="3" fill="1" visible="no" active="yes"/>
 <layer number="47" name="Measures" color="7" fill="1" visible="no" active="yes"/>
-<layer number="48" name="Document" color="7" fill="1" visible="yes" active="yes"/>
+<layer number="48" name="Document" color="7" fill="1" visible="no" active="yes"/>
 <layer number="49" name="Reference" color="7" fill="1" visible="no" active="yes"/>
 <layer number="50" name="dxf" color="7" fill="1" visible="no" active="no"/>
@@
 </autorouter>
 <elements>
-<element name="U2" library="SparkFun-IC-Special-Function" library_urn="urn:adsk.eagle:library:527" package="TSSOP-28_4MM" package3d_urn="urn:adsk.eagle:package:39196/1" value="PCA9685" x="58.6552" y="73.0592" smashed="yes" rot="R90">
+<element name="U2" library="SparkFun-IC-Special-Function" package="TSSOP-28_4MM" value="PCA9685" x="58.6552" y="73.0592" smashed="yes" rot="R90">
 <attribute name="PROD_ID" value="IC-12271" x="58.6552" y="73.0592" size="1.778" layer="27" rot="R90" display="off"/>
 </element>
@@
 <attribute name="PROD_ID" value="CAP-08280" x="119.3528" y="59.5872" size="1.778" layer="27" rot="R180" display="off"/>
 </element>
-<element name="JP2" library="SparkFun-Connectors" package="JST-2-PTH" value="LiPo" x="105.532" y="68.8904" smashed="yes" rot="MR270">
-<attribute name="PROD_ID" value="CONN-09863" x="109.032" y="72.3904" size="1.778" layer="28" rot="MR270" display="off"/>
-<attribute name="SKU" value="PRT-09914" x="109.032" y="72.3904" size="1.778" layer="28" rot="MR270" display="off"/>
-</element>
+<element name="JP2" library="SparkFun-Connectors" package="JST-2-PTH-NS" value="LiPo" x="105.532" y="68.8904" smashed="yes" rot="MR270"/>
 <element name="D1" library="SparkFun-LED" package="LED-0603" value="Yellow" x="114.2336" y="77.9744" smashed="yes" rot="R180">
 <attribute name="PROD_ID" value="DIO-09003" x="132.7336" y="70.9744" size="1.778" layer="27" rot="R180" display="off"/>
@@
 <attribute name="TP_SIGNAL_NAME" value="" x="107.554" y="77.3176" size="1" layer="38" rot="MR0"/>
 <attribute name="VALUE" x="108.316" y="78.9686" size="0.0254" layer="28" rot="MR0"/>
+</element>
+<element name="R5" library="SparkFun-Resistors" package="0603" value="3k" x="114.1856" y="76.96" smashed="yes" rot="MR90">
+<attribute name="PROD_ID" value="RES-08296" x="114.1856" y="76.96" size="1.778" layer="28" rot="MR90" display="off"/>
+</element>
+<element name="R7" library="SparkFun-Resistors" package="0603" value="1k" x="105.7968" y="78" smashed="yes" rot="MR180">
+<attribute name="PROD_ID" value="RES-08296" x="105.7968" y="78" size="1.778" layer="28" rot="MR180" display="off"/>
 </element>
 </elements>
@@
 <contactref element="SHOULDER01" pad="P$18"/>
 <contactref element="TO_SHOULDER01" pad="P$18"/>
-<contactref element="TP2" pad="TP"/>
+<contactref element="R5" pad="1"/>
 <wire x1="88" y1="55" x2="86" y2="55" width="0" layer="19" extent="16-16"/>
 <wire x1="96.012" y1="83.058" x2="93" y2="83" width="0" layer="19" extent="16-16"/>
@@
 <wire x1="53" y1="73.85" x2="54.4302" y2="75.2802" width="0.4064" layer="1"/>
 <wire x1="54.4302" y1="75.2802" x2="54.4302" y2="75.4614" width="0.4064" layer="1"/>
-<wire x1="89" y1="56.8468" x2="108.51530625" y2="61.824396875" width="0" layer="19" extent="16-16"/>
+<contactref element="R7" pad="1"/>
+<wire x1="104.9468" y1="78" x2="104.918" y2="78.0288" width="0.1524" layer="16"/>
+<wire x1="104.918" y1="78.0288" x2="104.0384" y2="78.0288" width="0.1524" layer="16"/>
+<via x="104.0384" y="78.0288" extent="1-16" drill="0.2"/>
+<wire x1="89.0524" y1="80.3416" x2="104.0384" y2="78.0288" width="0" layer="19" extent="16-16"/>
 <wire x1="78.0288" y1="57.0992" x2="88.4936" y2="57.3532" width="0" layer="19" extent="16-16"/>
 <wire x1="58.484690625" y1="61.824396875" x2="78" y2="57.0704" width="0" layer="19" extent="16-16"/>
@@
 <wire x1="113.792" y1="79" x2="113.792" y2="78.1812" width="0.2032" layer="16"/>
 <wire x1="113.792" y1="78.1812" x2="113.9952" y2="77.978" width="0.2032" layer="16"/>
-<wire x1="113.9952" y1="77.978" x2="115.0112" y2="77.978" width="0.2032" layer="16"/>
+<wire x1="113.9952" y1="77.978" x2="114.4016" y2="77.978" width="0.2032" layer="16"/>
 <contactref element="TP1" pad="TP"/>
+<wire x1="114.4016" y1="77.978" x2="115.0112" y2="77.978" width="0.2032" layer="16"/>
 <wire x1="113.554" y1="79.8576" x2="113.792" y2="79.6196" width="0.2" layer="16"/>
 <wire x1="113.792" y1="79.6196" x2="113.792" y2="79" width="0.2" layer="16"/>
+<contactref element="R5" pad="2"/>
+<wire x1="114.1856" y1="77.81" x2="114.2336" y2="77.81" width="0.1524" layer="16"/>
+<wire x1="114.2336" y1="77.81" x2="114.4016" y2="77.978" width="0.1524" layer="16"/>
+</signal>
+<signal name="N$42">
+<contactref element="TP2" pad="TP"/>
+<contactref element="R7" pad="2"/>
+<wire x1="107.554" y1="79.8576" x2="107.554" y2="78.9072" width="0.1524" layer="16"/>
+<wire x1="107.554" y1="78.9072" x2="106.6468" y2="78" width="0.1524" layer="16"/>
 </signal>
 </signals>

Commit message: REVIEW2010230495094059 Signed-off-by: Julian <julian.wingert@subtilitas.de>
Parts:
- moved U$1 1.70 mm to (52.0, 74.7)
- moved U$2 1.70 mm to (115.0, 72.7)
Routing:
- net V_USB: track 32.8 -> 40.6 mm
- net GND: track 29.5 -> 31.5 mm, vias 75 -> 78
- net FW_RST: track 13.6 -> 11.8 mm
- net TXD: track 14.9 -> 13.2 mm
- net SDA: track 51.3 -> 53.0 mm
- net RXD: track 16.2 -> 14.5 mm
- net SCL: track 50.3 -> 51.7 mm
Other:
- board size 69 x 38 mm -> 69 x 38.5 mm
