File: eaglefiles/crawler2body.brd (EAGLE design)
At the start: 69 x 38.5 mm, 45 parts, among them J2 USB-AB-MICROB-2, U1 MCP73831, U2 PCA9685, U3 FT232R, U5 LM3671MF-3.3/NOPB

Commit message: ORDERED VERSION!!!!11elf Signed-off-by: Julian <julian.wingert@subtilitas.de>
Parts:
- added R8, R9: 3k, SparkFun-Resistors:0603
Connections:
- net +3V3: now also R8.2, R9.2
- net SCL: now also R9.1
- net SDA: now also R8.1
Routing:
- net +3V3: track 24.8 -> 28.4 mm, vias 9 -> 10
- net SCL: track 51.7 -> 52.3 mm
