File: eaglefiles/crawler2body.sch (EAGLE design)
At the start: 40 parts, among them J2 USB-AB-MICROB-2, U1 MCP73831, U2 PCA9685, U3 FT232R, U5 LM3671MF-3.3/NOPB

Commit message: review 2
Signed-off-by: Julian <julian.wingert@subtilitas.de>
Parts:
- added TP1, TP2: PTR1TP15SQ, testpad:PTR1TP15SQ
- added U$8: MF-SMDF150, fuse:MF-SMDF150
Connections:
- removed net N$42: U$2.P$10
- new net FW_RST: TP1.TP, U$2.P$10
- new net N$46: JP2.2, U$8.1
- net +3V3: no longer U3.VCCIO
- net 3.3VFTDI: now also U3.VCCIO
- net GND: now also TP2.TP
- net USB_D+: now also J2.D+; no longer J2.D-
- net USB_D-: now also J2.D-; no longer J2.D+
- net V+: now also U$8.2; no longer JP2.2
Other:
- note removed: "SJ1 can be cut to modify the charge- current programming resistor."
- moved on the sheet: JP2

Commit message: Review-review-review Signed-off-by: Julian <julian.wingert@subtilitas.de>
Parts:
- added R5: 3k, SparkFun-Resistors:2.0KOHM1/10W5%(0603)
- added R7: 1k, SparkFun-Resistors:2.0KOHM1/10W5%(0603)
- JP2: device SparkFun-Connectors:M02JST-PTH-2 -> SparkFun-Connectors:M02-JST-2-PTH-NO_SILK
Connections:
- new net N$42: R7.2, TP2.TP
- net +3V3: now also R7.1
- net FW_RST: now also R5.2
- net GND: now also R5.1; no longer TP2.TP
Changed lines of the file:
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@@
 </classes>
 <parts>
-<part name="U2" library="SparkFun-IC-Special-Function" library_urn="urn:adsk.eagle:library:527" deviceset="PCA9685" device="" package3d_urn="urn:adsk.eagle:package:39196/1" value="PCA9685"/>
+<part name="U2" library="SparkFun-IC-Special-Function" deviceset="PCA9685" device="" value="PCA9685"/>
 <part name="GND2" library="supply1" library_urn="urn:adsk.eagle:library:371" deviceset="GND" device=""/>
 <part name="GND3" library="supply1" library_urn="urn:adsk.eagle:library:371" deviceset="GND" device=""/>
@@
 <part name="GND12" library="SparkFun-Aesthetics" deviceset="GND" device=""/>
 <part name="C6" library="SparkFun-Capacitors" deviceset="4.7UF" device="0603" value="4.7uF"/>
-<part name="JP2" library="SparkFun-Connectors" deviceset="M02" device="JST-PTH-2" value="LiPo"/>
+<part name="JP2" library="SparkFun-Connectors" deviceset="M02" device="-JST-2-PTH-NO_SILK" value="LiPo"/>
 <part name="GND7" library="SparkFun-Aesthetics" deviceset="GND" device=""/>
 <part name="D1" library="SparkFun-LED" deviceset="LED-YELLOW" device="0603" value="Yellow"/>
@@
 <part name="C10" library="rcl" library_urn="urn:adsk.eagle:library:334" deviceset="C-EU" device="C1210" package3d_urn="urn:adsk.eagle:package:23619/2" value="1uF"/>
 <part name="U$8" library="fuse" library_urn="urn:adsk.eagle:library:233" deviceset="MF-SMDF" device="" package3d_urn="urn:adsk.eagle:package:14081/1" technology="150"/>
-<part name="GND26" library="supply1" library_urn="urn:adsk.eagle:library:371" deviceset="GND" device=""/>
 <part name="TP1" library="testpad" library_urn="urn:adsk.eagle:library:385" deviceset="PTR1" device="TP15SQ" package3d_urn="urn:adsk.eagle:package:27975/1" value="PTR1TP15SQ"/>
 <part name="TP2" library="testpad" library_urn="urn:adsk.eagle:library:385" deviceset="PTR1" device="TP15SQ" package3d_urn="urn:adsk.eagle:package:27975/1" value="PTR1TP15SQ"/>
+<part name="+3V13" library="supply1" deviceset="+3V3" device=""/>
+<part name="R5" library="SparkFun-Resistors" deviceset="2.0KOHM1/10W5%(0603)" device="" value="3k"/>
+<part name="GND26" library="SparkFun-Aesthetics" deviceset="GND" device=""/>
+<part name="R7" library="SparkFun-Resistors" deviceset="2.0KOHM1/10W5%(0603)" device="" value="1k"/>
 </parts>
 <sheets>
@@
 <instance part="C10" gate="G$1" x="339.09" y="81.28"/>
 <instance part="U$8" gate="A" x="-57.15" y="198.12"/>
-<instance part="GND26" gate="1" x="138.43" y="210.82"/>
 <instance part="TP1" gate="G$1" x="116.84" y="210.82"/>
 <instance part="TP2" gate="G$1" x="132.08" y="210.82"/>
+<instance part="+3V13" gate="G$1" x="147.32" y="223.52"/>
+<instance part="R5" gate="G$1" x="102.87" y="208.28" rot="MR90"/>
+<instance part="GND26" gate="1" x="102.87" y="195.58" rot="MR0"/>
+<instance part="R7" gate="G$1" x="142.24" y="213.36" rot="MR0"/>
 </instances>
 <busses>
@@
 </segment>
 <segment>
+<pinref part="R5" gate="G$1" pin="1"/>
 <pinref part="GND26" gate="1" pin="GND"/>
-<wire x1="138.43" y1="213.36" x2="132.08" y2="213.36" width="0.1524" layer="91"/>
-<pinref part="TP2" gate="G$1" pin="TP"/>
+<wire x1="102.87" y1="198.12" x2="102.87" y2="203.2" width="0.1524" layer="91"/>
 </segment>
 </net>
@@
 <wire x1="264.16" y1="182.88" x2="281.94" y2="182.88" width="0.1524" layer="91"/>
 <pinref part="TO_HIP02" gate="G$1" pin="P$14"/>
+</segment>
+<segment>
+<pinref part="R7" gate="G$1" pin="1"/>
+<pinref part="+3V13" gate="G$1" pin="+3V3"/>
+<wire x1="147.32" y1="220.98" x2="147.32" y2="213.36" width="0.1524" layer="91"/>
 </segment>
 </net>
@@
 </segment>
 <segment>
-<wire x1="116.84" y1="213.36" x2="110.49" y2="213.36" width="0.1524" layer="91"/>
-<label x="110.49" y="213.36" size="1.27" layer="95" rot="R180" xref="yes"/>
+<wire x1="116.84" y1="213.36" x2="102.87" y2="213.36" width="0.1524" layer="91"/>
+<label x="93.98" y="213.36" size="1.27" layer="95" rot="R180" xref="yes"/>
 <pinref part="TP1" gate="G$1" pin="TP"/>
-</segment>
-</net>
+<pinref part="R5" gate="G$1" pin="2"/>
+<wire x1="102.87" y1="213.36" x2="93.98" y2="213.36" width="0.1524" layer="91"/>
+<junction x="102.87" y="213.36"/>
+</segment>
+</net>
+<net name="N$42" class="0">
+<segment>
+<pinref part="TP2" gate="G$1" pin="TP"/>
+<pinref part="R7" gate="G$1" pin="2"/>
+<wire x1="137.16" y1="213.36" x2="132.08" y2="213.36" width="0.1524" layer="91"/>
+</segment>
+</net>

Commit message: ORDERED VERSION!!!!11elf Signed-off-by: Julian <julian.wingert@subtilitas.de>
Parts:
- added R8, R9: 3k, SparkFun-Resistors:2.0KOHM1/10W5%(0603)
Connections:
- net +3V3: now also R8.2, R9.2
- net SCL: now also R9.1
- net SDA: now also R8.1
Changed lines of the file:
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@@
 <part name="GND26" library="SparkFun-Aesthetics" deviceset="GND" device=""/>
 <part name="R7" library="SparkFun-Resistors" deviceset="2.0KOHM1/10W5%(0603)" device="" value="1k"/>
+<part name="R8" library="SparkFun-Resistors" deviceset="2.0KOHM1/10W5%(0603)" device="" value="3k"/>
+<part name="R9" library="SparkFun-Resistors" deviceset="2.0KOHM1/10W5%(0603)" device="" value="3k"/>
 </parts>
 <sheets>
@@
 <instance part="GND26" gate="1" x="102.87" y="195.58" rot="MR0"/>
 <instance part="R7" gate="G$1" x="142.24" y="213.36" rot="MR0"/>
+<instance part="R8" gate="G$1" x="52.07" y="43.18" rot="MR90"/>
+<instance part="R9" gate="G$1" x="59.69" y="43.18" rot="MR90"/>
 </instances>
 <busses>
@@
 </segment>
 <segment>
-<wire x1="76.2" y1="31.75" x2="67.31" y2="31.75" width="0.1524" layer="91"/>
-<label x="67.31" y="31.75" size="1.016" layer="95" rot="R180" xref="yes"/>
+<wire x1="76.2" y1="31.75" x2="52.07" y2="31.75" width="0.1524" layer="91"/>
+<label x="52.07" y="31.75" size="1.016" layer="95" rot="R180" xref="yes"/>
 <pinref part="U$2" gate="G$1" pin="P$1"/>
+<pinref part="R8" gate="G$1" pin="1"/>
+<wire x1="52.07" y1="38.1" x2="52.07" y2="31.75" width="0.1524" layer="91"/>
 </segment>
 <segment>
@@
 </segment>
 <segment>
-<wire x1="76.2" y1="34.29" x2="67.31" y2="34.29" width="0.1524" layer="91"/>
-<label x="67.31" y="34.29" size="1.016" layer="95" rot="R180" xref="yes"/>
+<wire x1="76.2" y1="34.29" x2="59.69" y2="34.29" width="0.1524" layer="91"/>
+<label x="59.69" y="34.29" size="1.016" layer="95" rot="R180" xref="yes"/>
 <pinref part="U$2" gate="G$1" pin="P$2"/>
+<pinref part="R9" gate="G$1" pin="1"/>
+<wire x1="59.69" y1="38.1" x2="59.69" y2="34.29" width="0.1524" layer="91"/>
 </segment>
 <segment>
@@
 <wire x1="69.85" y1="67.31" x2="69.85" y2="82.55" width="0.1524" layer="91"/>
 <pinref part="+3V1" gate="G$1" pin="+3V3"/>
-</segment>
-<segment>
+<pinref part="R8" gate="G$1" pin="2"/>
+<pinref part="R9" gate="G$1" pin="2"/>
+<wire x1="52.07" y1="48.26" x2="59.69" y2="48.26" width="0.1524" layer="91"/>
+<wire x1="59.69" y1="48.26" x2="59.69" y2="67.31" width="0.1524" layer="91"/>
+<wire x1="59.69" y1="67.31" x2="69.85" y2="67.31" width="0.1524" layer="91"/>
+<junction x="59.69" y="48.26"/>
+<junction x="69.85" y="67.31"/>
+</segment>
+<segment>
